File: HPB-01.kicad_sch (KiCad schematic)
At the start: 62 parts, among them J1 USB_A, J4 USB_C_Receptacle_USB2.0, J5 Pad, J6 Pad, J7 Battery Pad, J8 Battery Pad, Q1 RU207C, Q4 RU20P7C, Q5 IRF7832, Q6 IRF7832, SW1 SW_Push, U1 S-8261ABJMD-G3JT2S, U2 IP5328P

Commit message: revision 1.1
Parts:
- removed C18, C24: 22uF, Capacitor_SMD:C_0805_2012Metric, symbol Device:C_Small
- C15, C17, C19, C21, C25, C3: value 10uF -> 22uF; footprint Capacitor_SMD:C_1206_3216Metric -> Capacitor_SMD:C_0805_2012Metric; LCSC C13585 -> C45783
- H1, H2, H3, H4: now left out of the parts list
Changed lines of the file:
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@@
-    (stroke (width 0) (type default) (color 0 0 0 0))
-  )
-  (wire (pts (xy 194.31 17.78) (xy 194.31 26.67))
     (stroke (width 0) (type default) (color 0 0 0 0))
   )
@@
   )
   (symbol (lib_id "Mechanical:MountingHole") (at 157.48 185.42 0) (unit 1)
-    (in_bom yes) (on_board yes) (fields_autoplaced)
+    (in_bom no) (on_board yes) (fields_autoplaced)
     (property "Reference" "H3" (id 0) (at 161.29 184.1499 0)
       (effects (font (size 1.27 1.27)) (justify left))
@@
   )
   (symbol (lib_id "Mechanical:MountingHole") (at 157.48 190.5 0) (unit 1)
-    (in_bom yes) (on_board yes) (fields_autoplaced)
+    (in_bom no) (on_board yes) (fields_autoplaced)
     (property "Reference" "H4" (id 0) (at 161.29 189.2299 0)
       (effects (font (size 1.27 1.27)) (justify left))
@@
   )
   (symbol (lib_id "Mechanical:MountingHole") (at 157.48 180.34 0) (unit 1)
-    (in_bom yes) (on_board yes) (fields_autoplaced)
+    (in_bom no) (on_board yes) (fields_autoplaced)
     (property "Reference" "H2" (id 0) (at 161.29 179.0699 0)
       (effects (font (size 1.27 1.27)) (justify left))
@@
       (effects (font (size 1.27 1.27)) (justify left))
     )
-    (property "Value" "10uF" (id 1) (at 280.67 77.4762 0)
-      (effects (font (size 1.27 1.27)) (justify left))
-    )
-    (property "Footprint" "Capacitor_SMD:C_1206_3216Metric" (id 2) (at 278.13 76.2 0)
+    (property "Value" "22uF" (id 1) (at 280.67 77.4762 0)
+      (effects (font (size 1.27 1.27)) (justify left))
+    )
+    (property "Footprint" "Capacitor_SMD:C_0805_2012Metric" (id 2) (at 278.13 76.2 0)
       (effects (font (size 1.27 1.27)) hide)
     )
@@
       (effects (font (size 1.27 1.27)) hide)
     )
-    (property "LCSC" "C13585" (id 4) (at 278.13 76.2 0)
+    (property "LCSC" "C45783" (id 4) (at 278.13 76.2 0)
       (effects (font (size 1.27 1.27)) hide)
     )
@@
     (pin "2")
   )
-  (symbol (lib_id "Device:C_Small") (at 134.62 81.28 0) (unit 1)
-    (in_bom yes) (on_board yes) (fields_autoplaced)
-    (property "Reference" "C24" (id 0) (at 137.16 80.0099 0)
-      (effects (font (size 1.27 1.27)) (justify left))
-    )
-    (property "Value" "22uF" (id 1) (at 137.16 82.5499 0)
-      (effects (font (size 1.27 1.27)) (justify left))
-    )
-    (property "Footprint" "Capacitor_SMD:C_0805_2012Metric" (id 2) (at 134.62 81.28 0)
-      (effects (font (size 1.27 1.27)) hide)
-    )
-    (property "Datasheet" "~" (id 3) (at 134.62 81.28 0)
-      (effects (font (size 1.27 1.27)) hide)
-    )
-    (property "LCSC" "C45783" (id 4) (at 134.62 81.28 0)
-      (effects (font (size 1.27 1.27)) hide)
-    )
-    (pin "1")
-    (pin "2")
-  )
   (symbol (lib_id "Device:C_Small") (at 219.71 27.94 0) (unit 1)
     (in_bom yes) (on_board yes) (fields_autoplaced)
@@
       (effects (font (size 1.27 1.27)) (justify left))
     )
-    (property "Value" "10uF" (id 1) (at 234.95 80.0162 0)
-      (effects (font (size 1.27 1.27)) (justify left))
-    )
-    (property "Footprint" "Capacitor_SMD:C_1206_3216Metric" (id 2) (at 232.41 78.74 0)
+    (property "Value" "22uF" (id 1) (at 234.95 80.0162 0)
+      (effects (font (size 1.27 1.27)) (justify left))
+    )
+    (property "Footprint" "Capacitor_SMD:C_0805_2012Metric" (id 2) (at 232.41 78.74 0)
       (effects (font (size 1.27 1.27)) hide)
     )
@@
       (effects (font (size 1.27 1.27)) hide)
     )
-    (property "LCSC" "C13585" (id 4) (at 232.41 78.74 0)
+    (property "LCSC" "C45783" (id 4) (at 232.41 78.74 0)
       (effects (font (size 1.27 1.27)) hide)
     )
@@
       (effects (font (size 1.27 1.27)) (justify left))
     )
-    (property "Value" "10uF" (id 1) (at 246.38 77.4762 0)
-      (effects (font (size 1.27 1.27)) (justify left))
-    )
-    (property "Footprint" "Capacitor_SMD:C_1206_3216Metric" (id 2) (at 243.84 76.2 0)
+    (property "Value" "22uF" (id 1) (at 246.38 77.4762 0)
+      (effects (font (size 1.27 1.27)) (justify left))
+    )
+    (property "Footprint" "Capacitor_SMD:C_0805_2012Metric" (id 2) (at 243.84 76.2 0)
       (effects (font (size 1.27 1.27)) hide)
     )
@@
       (effects (font (size 1.27 1.27)) hide)
     )
-    (property "LCSC" "C13585" (id 4) (at 243.84 76.2 0)
+    (property "LCSC" "C45783" (id 4) (at 243.84 76.2 0)
       (effects (font (size 1.27 1.27)) hide)
     )
@@
   )
   (symbol (lib_id "Mechanical:MountingHole") (at 157.48 175.26 0) (unit 1)
-    (in_bom yes) (on_board yes) (fields_autoplaced)
+    (in_bom no) (on_board yes) (fields_autoplaced)
     (property "Reference" "H1" (id 0) (at 161.29 173.9899 0)
       (effects (font (size 1.27 1.27)) (justify left))
@@
       (effects (font (size 1.27 1.27)) hide)
     )
-  )
-  (symbol (lib_id "Device:C_Small") (at 127 100.33 0) (unit 1)
-    (in_bom yes) (on_board yes) (fields_autoplaced)
-    (property "Reference" "C18" (id 0) (at 129.54 99.0599 0)
-      (effects (font (size 1.27 1.27)) (justify left))
-    )
-    (property "Value" "22uF" (id 1) (at 129.54 101.5999 0)
-      (effects (font (size 1.27 1.27)) (justify left))
-    )
-    (property "Footprint" "Capacitor_SMD:C_0805_2012Metric" (id 2) (at 127 100.33 0)
-      (effects (font (size 1.27 1.27)) hide)
-    )
-    (property "Datasheet" "~" (id 3) (at 127 100.33 0)
-      (effects (font (size 1.27 1.27)) hide)
-    )
-    (property "LCSC" "C45783" (id 4) (at 127 100.33 0)
-      (effects (font (size 1.27 1.27)) hide)
-    )
-    (pin "1")
-    (pin "2")
   )
   (symbol (lib_id "Device:C_Small") (at 194.31 151.13 0) (unit 1)
@@
       (effects (font (size 1.27 1.27)) (justify left))
     )
-    (property "Value" "10uF" (id 1) (at 262.89 77.4762 0)
-      (effects (font (size 1.27 1.27)) (justify left))
-    )
-    (property "Footprint" "Capacitor_SMD:C_1206_3216Metric" (id 2) (at 260.35 76.2 0)
+    (property "Value" "22uF" (id 1) (at 262.89 77.4762 0)
+      (effects (font (size 1.27 1.27)) (justify left))
+    )
+    (property "Footprint" "Capacitor_SMD:C_0805_2012Metric" (id 2) (at 260.35 76.2 0)
       (effects (font (size 1.27 1.27)) hide)
     )
@@
       (effects (font (size 1.27 1.27)) hide)
     )
-    (property "LCSC" "C13585" (id 4) (at 260.35 76.2 0)
+    (property "LCSC" "C45783" (id 4) (at 260.35 76.2 0)
       (effects (font (size 1.27 1.27)) hide)
     )
@@
       (effects (font (size 1.27 1.27)) (justify right))
     )
-    (property "Value" "10uF" (id 1) (at 251.46 85.0962 0)
+    (property "Value" "22uF" (id 1) (at 251.46 85.0962 0)
       (effects (font (size 1.27 1.27)) (justify right))
     )
-    (property "Footprint" "Capacitor_SMD:C_1206_3216Metric" (id 2) (at 254 83.82 0)
+    (property "Footprint" "Capacitor_SMD:C_0805_2012Metric" (id 2) (at 254 83.82 0)
       (effects (font (size 1.27 1.27)) hide)
     )
@@
       (effects (font (size 1.27 1.27)) hide)
     )
-    (property "LCSC" "C13585" (id 4) (at 254 83.82 0)
+    (property "LCSC" "C45783" (id 4) (at 254 83.82 0)
       (effects (font (size 1.27 1.27)) hide)
     )
@@
       (effects (font (size 1.27 1.27)) (justify left))
     )
-    (property "Value" "10uF" (id 1) (at 271.78 85.0962 0)
-      (effects (font (size 1.27 1.27)) (justify left))
-    )
-    (property "Footprint" "Capacitor_SMD:C_1206_3216Metric" (id 2) (at 269.24 83.82 0)
+    (property "Value" "22uF" (id 1) (at 271.78 85.0962 0)
+      (effects (font (size 1.27 1.27)) (justify left))
+    )
+    (property "Footprint" "Capacitor_SMD:C_0805_2012Metric" (id 2) (at 269.24 83.82 0)
       (effects (font (size 1.27 1.27)) hide)
     )
@@
       (effects (font (size 1.27 1.27)) hide)
     )
-    (property "LCSC" "C13585" (id 4) (at 269.24 83.82 0)
+    (property "LCSC" "C45783" (id 4) (at 269.24 83.82 0)
       (effects (font (size 1.27 1.27)) hide)
     )
@@
     )
     (path "/8555a4a0-3187-4478-ba74-a91c8f72c444"
-      (reference "C3") (unit 1) (value "10uF") (footprint "Capacitor_SMD:C_1206_3216Metric")
+      (reference "C3") (unit 1) (value "22uF") (footprint "Capacitor_SMD:C_0805_2012Metric")
     )
     (path "/968bab63-ea32-4245-bcf6-727047759b25"
@@
     )
     (path "/7e0f178d-33ce-49ff-a5db-57a6270e43f2"
-      (reference "C15") (unit 1) (value "10uF") (footprint "Capacitor_SMD:C_1206_3216Metric")
+      (reference "C15") (unit 1) (value "22uF") (footprint "Capacitor_SMD:C_0805_2012Metric")
     )
     (path "/d241961b-4771-4a53-aa2c-7e2aeaa31f55"
@@
     )
     (path "/cf524de6-100f-4c60-9250-115a09bd2ce2"
-      (reference "C17") (unit 1) (value "10uF") (footprint "Capacitor_SMD:C_1206_3216Metric")
-    )
-    (path "/b2173c96-14c4-4a5e-b4dc-75e2a0b2a386"
-      (reference "C18") (unit 1) (value "22uF") (footprint "Capacitor_SMD:C_0805_2012Metric")
+      (reference "C17") (unit 1) (value "22uF") (footprint "Capacitor_SMD:C_0805_2012Metric")
     )
     (path "/cb4bd2e0-ad75-422e-9188-6de1fe3f0773"
-      (reference "C19") (unit 1) (value "10uF") (footprint "Capacitor_SMD:C_1206_3216Metric")
+      (reference "C19") (unit 1) (value "22uF") (footprint "Capacitor_SMD:C_0805_2012Metric")
     )
     (path "/c8816297-1a77-4ab9-8b2a-4cdc1ba44561"
@@
     )
     (path "/ddd62814-5d3d-4a22-80b6-4c3b5efa5d5a"
-      (reference "C21") (unit 1) (value "10uF") (footprint "Capacitor_SMD:C_1206_3216Metric")
+      (reference "C21") (unit 1) (value "22uF") (footprint "Capacitor_SMD:C_0805_2012Metric")
     )
     (path "/c605a9d7-e92a-4385-8413-d38cc66cf8de"
@@
       (reference "C23") (unit 1) (value "22uF") (footprint "Capacitor_SMD:C_0805_2012Metric")
     )
-    (path "/72bb3420-14a8-4955-aadd-7cd461409e43"
-      (reference "C24") (unit 1) (value "22uF") (footprint "Capacitor_SMD:C_0805_2012Metric")
-    )
     (path "/5eb71981-196f-422e-9ade-76ad533cd986"
-      (reference "C25") (unit 1) (value "10uF") (footprint "Capacitor_SMD:C_1206_3216Metric")
+      (reference "C25") (unit 1) (value "22uF") (footprint "Capacitor_SMD:C_0805_2012Metric")
     )
     (path "/db673549-1a6b-4ea1-b496-060591420e98"
